File: stm32f437vg.kicad_pcb (KiCad board)
At the start: 2 copper layers, 49 parts, among them P1 CONN_BOOT0, P10 CONN_01X17, P11 CONN_01X24, P12 Power 3.3V, P13 CONN_01X21, P14 USB_OTG, P15 CONN_02X03, P16 USB_A, P17 CONN_01X13, P18 CONN_01X05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

Commit message: pcb done
Parts:
- removed P11: CONN_01X24, Pin_Headers:Pin_Header_Straight_1x24
- added P20: CONN_01X03, Pin_Headers:Pin_Header_Straight_1x03, F.Cu at (111.1, 131.6)
- added P21: CONN_01X20, Pin_Headers:Pin_Header_Straight_1x20, F.Cu at (168.1, 131.6)
- added P22: PA3, Pin_Headers:Pin_Header_Straight_1x01, F.Cu at (115.4, 131.6)
- P4: value CONN_01X02 -> swd; footprint Pin_Headers:Pin_Header_Straight_1x02 -> Pin_Headers:Pin_Header_Straight_1x03
- moved P8 82.7 mm to (126.0, 68.2), turned to 90 degrees
- moved C15 82.1 mm to (152.9, 95.0), turned to 90 degrees
- moved C1 70.1 mm to (178.3, 72.6), turned to 270 degrees
- moved P4 63.9 mm to (175.2, 71.6)
- moved P14 61.9 mm to (193.3, 111.9)
- moved P1 60.2 mm to (122.3, 71.8), turned to 180 degrees
- moved P18 57.7 mm to (184.2, 94.5)
- moved C5 56.3 mm to (115.3, 110.7), turned to 270 degrees
- moved C18 55.4 mm to (180.8, 86.6), turned to 270 degrees
- moved P16 53.7 mm to (184.2, 85.6)
- moved R1 52.9 mm to (118.8, 67.8), turned to 90 degrees
- moved C8 51.7 mm to (155.6, 95.1), turned to 90 degrees
- moved C10 51.7 mm to (191.4, 121.2)
- moved D1 51.5 mm to (116.3, 68.6)
- moved P9 51.4 mm to (127.5, 135.3)
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Connections:
- C18 pad 2: Net-(C18-Pad2) -> GND
- C19 pad 2: Net-(C18-Pad2) -> GND
- P12 pad 1: GND -> Net-(P12-Pad1)
- P12 pad 2: Net-(P12-Pad2) -> Net-(P12-Pad1)
- P15 pad 3: Net-(P12-Pad2) -> Net-(P12-Pad1)
- P3 pad 1: Net-(P3-Pad1) -> Net-(C5-Pad2)
- P3 pad 3: Net-(C5-Pad2) -> Net-(C4-Pad1)
- P3 pad 4: Net-(P3-Pad4) -> GND
- P3 pad 5: Net-(C4-Pad1) -> Net-(P3-Pad5)
- P4 pad 2: Net-(P4-Pad2) -> GND
- U1 pad 7: Net-(P3-Pad1) -> Net-(P3-Pad5)
- U1 pad 72: Net-(P4-Pad2) -> Net-(P4-Pad3)
Routing:
- net GND: track 0.00 -> 639.1 mm
- net +3V3: track 0.00 -> 366.8 mm
- net +5V: track 0.00 -> 86.4 mm
- net Net-(P13-Pad19): track 0.00 -> 56.5 mm
- net Net-(P13-Pad18): track 0.00 -> 54.9 mm
- net Net-(P2-Pad5): track 0.00 -> 49.8 mm
- net Net-(P2-Pad4): track 0.00 -> 47.7 mm
- net Net-(P2-Pad3): track 0.00 -> 45.8 mm
- net Net-(D1-Pad2): track 0.00 -> 44.2 mm
- net Net-(P2-Pad2): track 0.00 -> 43.9 mm
- net Net-(P13-Pad1): track 0.00 -> 43.2 mm
- net Net-(P2-Pad1): track 0.00 -> 42.4 mm
- net Net-(P13-Pad2): track 0.00 -> 42.4 mm
- net Net-(P6-Pad1): track 0.00 -> 39.5 mm
- net Net-(C1-Pad1): track 0.00 -> 38.9 mm
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Other:
- board outline added: 106.9 x 74.1 mm

Commit message: pcb fix
Routing:
- net +3V3: track 366.8 -> 348.4 mm
- added copper zone on F.Cu, net GND
Other:
- board text added: "10 aug 2016"
- board text added: "Simple dev.board for STM32F437VGTx"
- board text added: "by Alexander Lutsai"
Changed lines of the file:
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@@
     (area 89.536199 65.152199 196.569401 139.419401)
     (thickness 1.6)
-    (drawings 9)
-    (tracks 654)
+    (drawings 12)
+    (tracks 646)
     (zones 0)
     (modules 51)
@@
   )
   (setup
-    (last_trace_width 0.25)
+    (last_trace_width 0.7)
     (user_trace_width 0.3)
     (user_trace_width 0.4)
@@
     (user_trace_width 1)
     (trace_clearance 0.2)
-    (zone_clearance 0.508)
+    (zone_clearance 0.25)
     (zone_45_only no)
     (trace_min 0.2)
@@
     )
   )
+  (gr_text "10 aug 2016" (at 97.9424 137.5664) (layer F.Cu)
+    (effects (font (size 1.5 1.5) (thickness 0.3)))
+  )
+  (gr_text "\nby Alexander Lutsai" (at 158.3436 134.7216) (layer F.Cu)
+    (effects (font (size 1.5 1.5) (thickness 0.3)))
+  )
+  (gr_text "Simple dev.board for STM32F437VGTx" (at 152.0952 68.3768) (layer F.Cu)
+    (effects (font (size 1.5 1.5) (thickness 0.3)))
+  )
   (dimension 106.8832 (width 0.3) (layer Dwgs.User)
     (gr_text "106,883 mm" (at 143.0528 55.6984) (layer Dwgs.User)
@@
   (segment (start 155.575 96.901) (end 155.575 96.123) (width 0.25) (layer F.Cu) (net 10))
   (segment (start 154.352 98.124) (end 155.575 96.901) (width 0.25) (layer F.Cu) (net 10))
+  (segment (start 179.07 136.906) (end 179.07 137.16) (width 0.7) (layer F.Cu) (net 11))
+  (segment (start 179.07 137.16) (end 178.2572 137.9728) (width 0.7) (layer F.Cu) (net 11))
+  (segment (start 179.07 129.921) (end 179.07 136.906) (width 0.7) (layer F.Cu) (net 11) (status 400000))
+  (segment (start 179.07 136.906) (end 179.07 137.0584) (width 0.7) (layer F.Cu) (net 11))
+  (segment (start 179.07 137.0584) (end 179.9844 137.9728) (width 0.7) (layer F.Cu) (net 11))
+  (segment (start 131.6736 137.9728) (end 178.2572 137.9728) (width 0.7) (layer F.Cu) (net 11))
+  (segment (start 117.2464 137.9728) (end 113.665 134.3914) (width 0.7) (layer F.Cu) (net 11))
+  (segment (start 131.6736 137.9728) (end 117.2464 137.9728) (width 0.7) (layer F.Cu) (net 11))
+  (segment (start 178.2572 137.9728) (end 179.9844 137.9728) (width 0.7) (layer F.Cu) (net 11))
+  (segment (start 179.9844 137.9728) (end 186.1058 137.9728) (width 0.7) (layer F.Cu) (net 11))
+  (segment (start 186.1058 137.9728) (end 190.373 133.7056) (width 0.7) (layer F.Cu) (net 11))
   (segment (start 135.9916 109.3724) (end 136.652 108.712) (width 0.7) (layer F.Cu) (net 11))
   (segment (start 145.2372 108.712) (end 136.652 108.712) (width 0.7) (layer F.Cu) (net 11))
   (segment (start 145.542 108.712) (end 145.2372 108.712) (width 0.25) (layer F.Cu) (net 11))
-  (segment (start 179.07 129.921) (end 179.07 136.3853) (width 0.7) (layer F.Cu) (net 11))
-  (segment (start 178.9176 136.4996) (end 178.9176 136.3853) (width 0.7) (layer F.Cu) (net 11))
-  (segment (start 178.9557 136.4996) (end 178.9176 136.4996) (width 0.7) (layer F.Cu) (net 11))
-  (segment (start 179.07 136.3853) (end 178.9557 136.4996) (width 0.7) (layer F.Cu) (net 11))
   (segment (start 91.7956 132.6388) (end 91.7956 102.1588) (width 0.7) (layer F.Cu) (net 11))
   (segment (start 113.665 134.3914) (end 93.5482 134.3914) (width 0.7) (layer F.Cu) (net 11))
   (segment (start 93.5482 134.3914) (end 91.7956 132.6388) (width 0.7) (layer F.Cu) (net 11))
-  (segment (start 187.5917 136.3853) (end 178.9176 136.3853) (width 0.7) (layer F.Cu) (net 11))
-  (segment (start 178.9176 136.3853) (end 133.2611 136.3853) (width 0.7) (layer F.Cu) (net 11))
-  (segment (start 133.2611 136.3853) (end 131.6736 137.9728) (width 0.7) (layer F.Cu) (net 11))
-  (segment (start 131.6736 137.9728) (end 117.2464 137.9728) (width 0.7) (layer F.Cu) (net 11))
-  (segment (start 117.2464 137.9728) (end 113.665 134.3914) (width 0.7) (layer F.Cu) (net 11))
   (segment (start 113.665 134.3914) (end 113.6396 134.366) (width 0.7) (layer F.Cu) (net 11))
-  (segment (start 190.373 133.7056) (end 190.2714 133.7056) (width 0.7) (layer F.Cu) (net 11))
-  (segment (start 190.2714 133.7056) (end 187.5917 136.3853) (width 0.7) (layer F.Cu) (net 11))
-  (segment (start 187.5917 136.3853) (end 187.579 136.398) (width 0.7) (layer F.Cu) (net 11))
   (segment (start 190.373 130.81) (end 190.373 133.7056) (width 0.7) (layer F.Cu) (net 11))
   (segment (start 190.373 133.7056) (end 190.373 135.2423) (width 0.7) (layer F.Cu) (net 11))
@@
   (segment (start 190.373 135.2423) (end 190.3857 135.255) (width 0.25) (layer F.Cu) (net 11))
   (segment (start 190.373 124.206) (end 190.373 130.81) (width 0.4) (layer F.Cu) (net 11))
-  (segment (start 179.07 129.921) (end 179.07 132.969) (width 0.25) (layer F.Cu) (net 11))
-  (segment (start 179.07 132.969) (end 179.07 134.62) (width 0.25) (layer F.Cu) (net 11))
-  (segment (start 179.07 134.62) (end 179.07 135.89) (width 0.25) (layer F.Cu) (net 11))
-  (segment (start 179.578 136.398) (end 187.579 136.398) (width 0.25) (layer F.Cu) (net 11))
-  (segment (start 179.07 135.89) (end 179.578 136.398) (width 0.25) (layer F.Cu) (net 11))
-  (segment (start 187.579 136.398) (end 190.373 133.604) (width 0.25) (layer F.Cu) (net 11))
-  (segment (start 190.373 133.604) (end 190.373 130.81) (width 0.25) (layer F.Cu) (net 11))
   (segment (start 116.84 134.366) (end 117.094 134.366) (width 0.25) (layer F.Cu) (net 11))
   (segment (start 115.062 134.366) (end 116.84 134.366) (width 0.25) (layer F.Cu) (net 11))
@@
   (segment (start 172.3136 81.5848) (end 172.3136 77.4192) (width 0.25) (layer F.Cu) (net 99))
   (segment (start 155.2744 98.624) (end 172.3136 81.5848) (width 0.25) (layer F.Cu) (net 99))
+  (zone (net 1) (net_name GND) (layer F.Cu) (hatch edge 0.508)
+    (connect_pads (clearance 0.25))
+    (min_thickness 0.254)
+    (fill (arc_segments 16) (thermal_gap 0.508) (thermal_bridge_width 0.508))
+    (polygon
+      (pts
+        (xy 89.6112 65.278) (xy 196.4944 65.278) (xy 196.4944 139.3444) (xy 89.6112 139.3444)
+      )
+    )
+  )
 )
